File: schematics/Arduino-xBee_shield_v1.kicad_pcb (KiCad board)
At the start: 2 copper layers, 39.4 x 87.6 mm, 5 parts, among them J1 Power In, J2 LX Serial, J3 xBee Serial

Commit message: gerber files
Parts:
- added REF**: MountingHole_2.2mm_M2, Mounting_Holes:MountingHole_2.2mm_M2, F.Cu at (168.3, 146.7)
- added REF**: MountingHole_2.2mm_M2, Mounting_Holes:MountingHole_2.2mm_M2, F.Cu at (135.3, 146.7)
- added REF**: MountingHole_2.2mm_M2, Mounting_Holes:MountingHole_2.2mm_M2, F.Cu at (156.8, 66.0)
- J2: value LX Serial -> LX
- J3: value xBee Serial -> xBee
- Power IN: renamed from J1
- renumbered Arduino1 to Arduino, xBee1 to xBee
Routing:
- net Net-(Arduino1-Pad3V3): track 120.0 -> 115.8 mm
Other:
- outline, holes or cut-outs redrawn
- board text added: "GND"
- board text added: "InciWinch Akaflieg Berlin"
- board text added: "Rx"
- board text added: "Tx"
- board text added: "Vin"
